File: pcb/Motherboard/motherboard.sch (EAGLE design)
At the start: 22 parts, among them U1 MIC5219 3.3V

Commit message: Added sensor board and reorganized
Parts:
- JP2, JP3: value M14 -> M13; device SparkFun-Connectors:M14 -> SparkFun-Connectors:M13
Connections:
- removed net PD5: JP2.14, U$1.PD5
- net PB4: now also JP3.10; no longer JP3.11
- net PB5: now also JP3.9; no longer JP3.10
- net PB6: now also JP3.8; no longer JP3.9
- net PC6: now also JP3.7; no longer JP3.8
- net PC7: now also JP3.6; no longer JP3.7
- net PD4: now also JP3.13; no longer JP3.14
- net PD6: now also JP3.12; no longer JP3.13
- net PD7: now also JP3.11; no longer JP3.12
- net PF0: no longer JP3.1
- net PF1: now also JP3.1; no longer JP3.2
- net PF4: now also JP3.2; no longer JP3.3
- net PF5: now also JP3.3; no longer JP3.4
- net PF6: now also JP3.4; no longer JP3.5
- net PF7: now also JP3.5; no longer JP3.6
